File: fan_breakout.kicad_sch (KiCad schematic)
At the start: 6 parts, among them J1 470531000, J2 470531000, J3 470531000, J4 TBL009-254-05GY-2GY

Commit message: Fix footprint links
Parts:
- J1, J2, J3: footprint CONN_SD-47053-001_H10p00_MOL -> footprints:molex_molex_470531000
- J4: footprint TBL009-254-05GY-2GY:CUI_TBL009-254-05GY-2GY -> footprints:Same_Sky_TBL009-254-05GY-2GY
Changed lines of the file:
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@@
 			)
 		)
-		(property "Footprint" "TBL009-254-05GY-2GY:CUI_TBL009-254-05GY-2GY"
+		(property "Footprint" "footprints:Same_Sky_TBL009-254-05GY-2GY"
 			(at 116.84 105.41 0)
 			(effects
@@
 			)
 		)
-		(property "Footprint" "CONN_SD-47053-001_H10p00_MOL"
+		(property "Footprint" "footprints:molex_molex_470531000"
 			(at 156.21 101.6 0)
 			(effects
@@
 			)
 		)
-		(property "Footprint" "CONN_SD-47053-001_H10p00_MOL"
+		(property "Footprint" "footprints:molex_molex_470531000"
 			(at 156.21 82.55 0)
 			(effects
@@
 			)
 		)
-		(property "Footprint" "CONN_SD-47053-001_H10p00_MOL"
+		(property "Footprint" "footprints:molex_molex_470531000"
 			(at 156.21 120.65 0)
 			(effects
